File: rc2014-512k-rom-ram.kicad_pcb (KiCad board)
At the start: 2 copper layers, 99.1 x 49.9 mm, 16 parts, among them J1 RC2014_Bus, U1 SST39SF040, U2 AS6C4008-55PCN, U3 74LS139, U4 74LS74, U5 74LS670, U6 74LS670, U7 74LS138

Commit message: Oops
Parts:
- moved C6 7.02 mm to (172.7, 91.4)
- moved U4 5.08 mm to (158.1, 108.6)
- moved C5 4.05 mm to (174.0, 95.9), turned to 180 degrees
Routing:
- net +5V: track 0.00 -> 221.7 mm, vias 0 -> 18
- net /ma18: track 0.00 -> 151.2 mm, vias 0 -> 7
- net /a14: track 0.00 -> 144.8 mm, vias 0 -> 7
- net /a15: track 0.00 -> 141.4 mm, vias 0 -> 6
- net /ma15: track 0.00 -> 117.8 mm, vias 0 -> 6
- net /a2: track 0.00 -> 116.5 mm, vias 0 -> 2
- net /ma14: track 0.00 -> 105.2 mm, vias 0 -> 5
- net /d4: track 0.00 -> 102.8 mm, vias 0 -> 6
- net /~{wr}: track 0.00 -> 100.4 mm, vias 0 -> 3
- net /a7: track 0.00 -> 100.2 mm, vias 0 -> 2
- net /a0: track 0.00 -> 98.4 mm, vias 0 -> 4
- net GND: track 0.00 -> 92.9 mm, vias 0 -> 9
- net /a6: track 0.00 -> 86.9 mm, vias 0 -> 3
- net /ma16: track 0.00 -> 86.8 mm, vias 0 -> 4
- net /~{mreq}: track 0.00 -> 82.8 mm, vias 0 -> 4
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- added copper zone on B.Cu, net GND

Commit message: Finally fully routed
Parts:
- removed C6: 0.1µF, Capacitor_THT:C_Disc_D4.7mm_W2.5mm_P5.00mm
- moved U3 19.3 mm to (179.1, 74.2), turned to 90 degrees
- moved RN1 0.76 mm to (172.7, 66.5)
- moved C2 0.64 mm to (109.9, 86.4)
Routing:
- net GND: track 92.9 -> 184.6 mm, vias 9 -> 11
- net /a1: track 58.0 -> 141.4 mm, vias 3 -> 6
- net /ma17: track 68.2 -> 146.1 mm, vias 2 -> 12
- net /ma16: track 86.8 -> 161.1 mm, vias 4 -> 7
- net /ma21: track 0.00 -> 73.0 mm, vias 0 -> 3
- net /a5: track 26.2 -> 97.2 mm, vias 0 -> 4
- net /~{wr}: track 100.4 -> 168.9 mm, vias 3 -> 6
- net /ma20: track 34.3 -> 92.5 mm, vias 0 -> 5
- net /d7: track 49.7 -> 100.8 mm, vias 2 -> 5
- net /a4: track 26.2 -> 74.8 mm, vias 0 -> 1
- net /ma15: track 117.8 -> 164.6 mm, vias 6 -> 4
- net /d6: track 47.3 -> 92.6 mm, vias 2 -> 5
- net /a0: track 98.4 -> 140.6 mm, vias 4 -> 7
- net /a14: track 144.8 -> 109.0 mm, vias 7 -> 4
- net /ma14: track 105.2 -> 140.1 mm
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- added copper zone on F.Cu, net +5V
Other:
- board text removed: "+5v"
- board text removed: "a0"
- board text removed: "a1"
- board text removed: "a10"
- board text removed: "a11"
- board text removed: "a12"
- board text removed: "a13"
- board text removed: "a14"
- board text removed: "a15"
- board text removed: "a2"
- board text removed: "a3"
- board text removed: "a4"
- board text removed: "a5"
- board text removed: "a6"
- board text removed: "a7"
- board text removed: "a8"
- board text removed: "a9"
- board text removed: "clk"
- board text removed: "d0"
- board text removed: "d1"
- board text removed: "d2"
- board text removed: "d3"
- board text removed: "d4"
- board text removed: "d5"
- board text removed: "d6"
- board text removed: "d7"
- board text removed: "gnd"
- board text removed: "rx"
- board text removed: "tx"
- board text removed: "user1"
- board text removed: "user2"
- board text removed: "user3"
- board text removed: "~{int}"
- board text removed: "~{iorq}"
- board text removed: "~{m1}"
- board text removed: "~{mreq}"
- board text removed: "~{rd}"
- board text removed: "~{reset}"
- board text removed: "~{wr}"

Commit message: labels
Routing:
- net /ma17: track 146.1 -> 144.7 mm
Other:
- board text added: "512k ROM/RAM for RC2014"
- board text added: "leadedsolder.com 2024 v1"
Changed lines of the file:
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@@
         (effects (font (size 1 1) (thickness 0.15)))
     )
-    (fp_text value "AS6C4008-55PCN" (at 10.795 41.275 90) (layer "F.SilkS")
+    (fp_text value "AS6C4008-55PCN" (at 8.382 41.489 90) (layer "F.SilkS")
         (effects (font (size 1 1) (thickness 0.15)))
     )
@@
     (property "ki_keywords" "R network star-topology")
     (attr through_hole)
-    (fp_text reference "RN1" (at 24.13 1.27) (layer "F.SilkS")
-        (effects (font (size 1 1) (thickness 0.15)))
-    )
-    (fp_text value "4.7kΩ" (at 24.765 -0.635) (layer "F.SilkS")
+    (fp_text reference "RN1" (at 8.382 -2.286) (layer "F.SilkS")
+        (effects (font (size 1 1) (thickness 0.15)))
+    )
+    (fp_text value "4.7kΩ" (at 20.32 -2.286) (layer "F.SilkS")
         (effects (font (size 1 1) (thickness 0.15)))
     )
@@
     (property "ki_keywords" "TTL Register 3State")
     (attr through_hole)
-    (fp_text reference "U6" (at 3.81 -2.33 90) (layer "F.SilkS")
+    (fp_text reference "U6" (at 4.445 -2.33 90) (layer "F.SilkS")
         (effects (font (size 1 1) (thickness 0.15)))
     )
@@
   (gr_line (start 201.31278 66.30162) (end 201.31278 68.24726)
     (stroke (width 0.2) (type solid)) (layer "F.CrtYd"))
+  (gr_text "leadedsolder.com 2024 v1" (at 119.634 69.088) (layer "F.Cu")
+    (effects (font (size 1.5 1.5) (thickness 0.3) bold) (justify left bottom))
+  )
+  (gr_text "512k ROM/RAM for RC2014" (at 118.618 66.802) (layer "F.Cu")
+    (effects (font (size 1.5 1.5) (thickness 0.3) bold) (justify left bottom))
+  )
   (gr_text "Pin 1" (at 105.26268 107.61218 90) (layer "F.SilkS")
     (effects (font (size 1.5 1.5) (thickness 0.3)))
+  )
+  (gr_text "512k ROM/RAM for RC2014" (at 118.618 66.802) (layer "F.Mask")
+    (effects (font (size 1.5 1.5) (thickness 0.3) bold) (justify left bottom))
+  )
+  (gr_text "leadedsolder.com 2024 v1" (at 119.634 69.088) (layer "F.Mask")
+    (effects (font (size 1.5 1.5) (thickness 0.3) bold) (justify left bottom))
   )
   (gr_text "135 deg" (at 121.73204 68.62064) (layer "F.CrtYd")
@@
   (segment (start 179.324 103.63145) (end 179.169868 103.477318) (width 0.45) (layer "F.Cu") (net 43))
   (segment (start 121.28 88.537412) (end 121.28 73.615) (width 0.45) (layer "F.Cu") (net 43))
-  (segment (start 120.055 72.39) (end 120.055 69.25555) (width 0.45) (layer "F.Cu") (net 43))
   (segment (start 192.024 108.331) (end 191.77 108.585) (width 0.45) (layer "F.Cu") (net 43))
   (segment (start 162.561 70.10445) (end 162.561 89.118808) (width 0.45) (layer "F.Cu") (net 43))
@@
   (segment (start 162.56 66.548) (end 162.56 69.596) (width 0.45) (layer "F.Cu") (net 43))
   (segment (start 162.56 69.596) (end 162.405868 69.750132) (width 0.45) (layer "F.Cu") (net 43))
-  (segment (start 120.055 69.25555) (end 120.042132 69.242682) (width 0.45) (layer "F.Cu") (net 43))
   (segment (start 185.928 103.175013) (end 185.791775 103.038788) (width 0.45) (layer "F.Cu") (net 43))
   (segment (start 186.088719 106.68) (end 185.928 106.519281) (width 0.45) (layer "F.Cu") (net 43))
+  (segment (start 120.055 70.67045) (end 120.76245 69.963) (width 0.45) (layer "F.Cu") (net 43))
   (segment (start 175.26 89.408) (end 175.26 100.076) (width 0.45) (layer "F.Cu") (net 43))
   (segment (start 175.613868 100.429868) (end 175.613868 103.477318) (width 0.45) (layer "F.Cu") (net 43))
+  (segment (start 120.055 72.39) (end 120.055 70.67045) (width 0.45) (layer "F.Cu") (net 43))
   (segment (start 175.26 100.076) (end 175.613868 100.429868) (width 0.45) (layer "F.Cu") (net 43))
   (segment (start 120.055 92.075) (end 120.055 89.762412) (width 0.45) (layer "F.Cu") (net 43))
@@
   (via (at 188.468 102.616) (size 0.8) (drill 0.4) (layers "F.Cu" "B.Cu") (net 43))
   (via (at 189.484 105.156) (size 0.8) (drill 0.4) (layers "F.Cu" "B.Cu") (net 43))
-  (via (at 120.042132 69.242682) (size 0.8) (drill 0.4) (layers "F.Cu" "B.Cu") (net 43))
+  (via (at 120.76245 69.963) (size 0.8) (drill 0.4) (layers "F.Cu" "B.Cu") (net 43))
   (segment (start 162.850192 89.408) (end 162.786 89.343808) (width 0.45) (layer "B.Cu") (net 43))
   (segment (start 160.003574 69.37) (end 160.582892 69.949318) (width 0.45) (layer "B.Cu") (net 43))
@@
   (segment (start 120.76245 69.963) (end 157.306523 69.963) (width 0.45) (layer "B.Cu") (net 43))
   (segment (start 175.26 89.408) (end 162.850192 89.408) (width 0.45) (layer "B.Cu") (net 43))
-  (segment (start 120.042132 69.242682) (end 120.76245 69.963) (width 0.45) (layer "B.Cu") (net 43))
   (segment (start 175.825186 103.266) (end 175.613868 103.477318) (width 0.45) (layer "B.Cu") (net 43))
   (segment (start 160.582892 69.949318) (end 162.405868 69.949318) (width 0.45) (layer "B.Cu") (net 43))
@@
   (via (at 177.023873 76.668) (size 0.8) (drill 0.4) (layers "F.Cu" "B.Cu") (net 44))
   (via (at 200.830984 84.20248) (size 0.8) (drill 0.4) (layers "F.Cu" "B.Cu") (net 44))
-  (segment (start 157.718762 70.47) (end 159.476257 70.47) (width 0.45) (layer "B.Cu") (net 44))
   (segment (start 176.129057 86.6) (end 175.104057 87.625) (width 0.45) (layer "B.Cu") (net 44))
-  (segment (start 159.476257 70.47) (end 159.701257 70.245) (width 0.45) (layer "B.Cu") (net 44))
-  (segment (start 114.301 70.613) (end 157.575761 70.613) (width 0.45) (layer "B.Cu") (net 44))
+  (segment (start 157.575761 70.613) (end 157.943761 70.245) (width 0.45) (layer "B.Cu") (net 44))
   (segment (start 177.248873 76.443) (end 177.023873 76.668) (width 0.45) (layer "B.Cu") (net 44))
-  (segment (start 113.792 70.104) (end 114.301 70.613) (width 0.45) (layer "B.Cu") (net 44))
   (segment (start 199.940504 83.312) (end 200.830984 84.20248) (width 0.45) (layer "B.Cu") (net 44))
-  (segment (start 157.575761 70.613) (end 157.718762 70.47) (width 0.45) (layer "B.Cu") (net 44))
+  (segment (start 113.792 70.104) (end 114.453 70.765) (width 0.45) (layer "B.Cu") (net 44))
+  (segment (start 121.349887 70.613) (end 157.575761 70.613) (width 0.45) (layer "B.Cu") (net 44))
+  (segment (start 121.124887 70.838) (end 121.349887 70.613) (width 0.45) (layer "B.Cu") (net 44))
+  (segment (start 157.943761 70.245) (end 159.701257 70.245) (width 0.45) (layer "B.Cu") (net 44))
+  (segment (start 120.562412 70.765) (end 120.635412 70.838) (width 0.45) (layer "B.Cu") (net 44))
   (segment (start 196.596 83.312) (end 199.940504 83.312) (width 0.45) (layer "B.Cu") (net 44))
+  (segment (start 120.635412 70.838) (end 121.124887 70.838) (width 0.45) (layer "B.Cu") (net 44))
   (segment (start 160.126 87.625) (end 159.512 87.011) (width 0.45) (layer "B.Cu") (net 44))
   (segment (start 175.104057 87.625) (end 160.126 87.625) (width 0.45) (layer "B.Cu") (net 44))
   (segment (start 200.830986 76.2) (end 200.587986 76.443) (width 0.45) (layer "B.Cu") (net 44))
+  (segment (start 114.453 70.765) (end 120.562412 70.765) (width 0.45) (layer "B.Cu") (net 44))
   (segment (start 200.587986 76.443) (end 177.248873 76.443) (width 0.45) (layer "B.Cu") (net 44))
   (segment (start 181.61 74.168) (end 181.61 70.358) (width 0.45) (layer "F.Cu") (net 45))
