File: rc2014-512k-rom-ram.kicad_pcb (KiCad board)
At the start: 2 copper layers, 99.1 x 49.9 mm, 16 parts, among them J1 RC2014_Bus, U1 SST39SF040, U2 AS6C4008-55PCN, U3 74LS139, U4 74LS74, U5 74LS670, U6 74LS670, U7 74LS138

Commit message: KiCad 9; fix designators
Parts:
- removed the REF** at (156.2, 78.2)
- renumbered U5 to U3, U6 to U4, U3 to U5, U4 to U6
